File: Esquema Fuente PLL/power_supply/power_supply.kicad_pcb (KiCad board)
At the start: 2 copper layers, 78 x 66.5 mm, 11 parts, among them J1 Terminal_01x02, J7 Terminal_01x02, J8 Terminal_01x03

Commit message: Se agrega pcb de crowbar
Parts:
- added D1: 1N4007, Diode_THT:D_DO-41_SOD81_P10.16mm_Horizontal, F.Cu at (166.4, 83.3)
- added D2: 1N4007, Diode_THT:D_DO-41_SOD81_P10.16mm_Horizontal, F.Cu at (166.4, 110.0)
- added D3: 4.7V, Diode_THT:D_DO-41_SOD81_P10.16mm_Horizontal, F.Cu at (173.0, 112.0)
- added D5: 12V, Diode_THT:D_DO-41_SOD81_P10.16mm_Horizontal, F.Cu at (173.0, 81.5)
- added D7: Q_SCR_KGA, Package_TO_SOT_THT:TO-92_Wide, F.Cu at (181.0, 105.0)
- added D8: Q_SCR_KGA, Package_TO_SOT_THT:TO-92L_Wide, F.Cu at (181.0, 87.0)
- added H5: MountingHole_2.2mm_M2_ISO7380_Pad, MountingHole:MountingHole_2.2mm_M2_ISO7380_Pad, F.Cu at (155.5, 79.2)
- added H6: MountingHole_2.2mm_M2_ISO7380_Pad, MountingHole:MountingHole_2.2mm_M2_ISO7380_Pad, F.Cu at (189.0, 79.2)
- added H7: MountingHole_2.2mm_M2_ISO7380_Pad, MountingHole:MountingHole_2.2mm_M2_ISO7380_Pad, F.Cu at (189.0, 113.0)
- added H8: MountingHole_2.2mm_M2_ISO7380_Pad, MountingHole:MountingHole_2.2mm_M2_ISO7380_Pad, F.Cu at (155.5, 113.0)
- added J2: 01x03, TerminalBlock:TerminalBlock_MaiXu_MX126-5.0-03P_1x03_P5.00mm, F.Cu at (157.5, 91.1)
- added R1: 100, Resistor_THT:R_Axial_DIN0207_L6.3mm_D2.5mm_P10.16mm_Horizontal, F.Cu at (173.9, 99.8)
- added R2: 100, Resistor_THT:R_Axial_DIN0207_L6.3mm_D2.5mm_P10.16mm_Horizontal, F.Cu at (173.9, 93.5)
- moved J1 52.6 mm to (104.3, 85.7)
- moved J7 52.6 mm to (104.3, 112.7)
- moved F1 52.6 mm to (38.2, 93.7)
- moved H1 52.6 mm to (37.2, 65.7)
- moved H4 52.6 mm to (37.2, 123.2)
- moved J8 52.6 mm to (38.2, 106.7)
- moved PS2 52.6 mm to (57.7, 110.7)
- moved PS3 52.6 mm to (57.7, 73.7)
- moved RV1 52.6 mm to (50.2, 73.7)
- moved H2 52.6 mm to (106.7, 65.7)
- moved H3 52.6 mm to (106.7, 123.2)
Routing:
- net +5V: track 20.9 -> 54.6 mm
- net +12V: track 13.0 -> 44.5 mm
- net Net-(D3-A): track 0.00 -> 20.7 mm
- net Net-(D5-A): track 0.00 -> 20.4 mm
Other:
- board size 78 x 66.5 mm -> 159.5 x 66.5 mm
